File: StepperServo.kicad_sch (KiCad schematic)
At the start: 21 parts, among them J1 Conn_01x01_Female, J2 Conn_01x01_Female, U1 TC1185, U2 SN65HVD232, U7 INA180A1

Commit message: Update notes
Other:
- note added: "Input Current: Voltage about 12V Motor: 8.08W Driver: 1.31W == Iin = (8.08W + 1.31W) / 12V = 0.78A"
- note added: "Power losses at TMC2209: From datasheet at 1A rms, 24V, Stealth Ploss = 1.4W Loss is internal LDO + Drive Stage LDO Current output = 7.5mA at 24V, 1A rms: LDO: 24V * 0.0075 = 0.18W Drive: (1.4W - 0.18W) / 1 A = 1,22 Ohm at 12V, 1A rms: LDO: 12V * 0.0075 = 0.09W Drive: 1A² * 1.22 Ohm = 1.22W = 1,31W loss at TMC2209 -----------------------------------"
- note added: "Power losses at motor: cheap Stepper motor 42HB34F1AB-01 as reference: - max 1 A phase current - 4 Ohm coil resistance -> 4V, 4W resistive losses - tear down: 5 - revolutions: 2 - goal time: 2.5 sec -> speed (5*2)/2.5 rps = 4 rps - holding torque: 0.23Nm Back emf approximation: (sqrt(2) * 3.14 * 0.23Nm * 4 1/s) / 1A = 4.08V = (4.08V bemf + 4V resistive loss) * 1A = 8.08W loss at motor -----------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"
- note removed: "Current (Worst Case): Battery low Voltage about 14.7V Motor: 3.8W Driver: 0.3W == Iin = 0.27A"
- note removed: "Power losses TMC2209: From datasheet at 1A rms, 24V, Stealth Ploss = 1.4W Loss is internal LDO + Drive Stage LDO Current output = 7.5mA at 24V, 1A rms: LDO: 24V * 0.0075 = 0.18W Drive: (1.4W - 0.18W) / 1 A = 1,22 Ohm at 16.8V, 0.4A rms: LDO: 16.8V * 0.0075 = 0.12W Drive: 0.4A² * 1.22 Ohm = 0.19W == Loss: 0,3W"
- note removed: "Stepper motor: 14HY2420 - used at 0.4 A phase current - 20 Ohm coil resistance -> 8V, 3.2W resistive losses - fast rc car servos do up to 80 rpm, 1.3 rps - match at least that - holding torque: 0.12Nm Back emf approximation: (sqrt(2) * 3.14 * 0.12Nm * 1.3 1/s *) / 0.4A = 1.7V == (1.7V bemf + 8V resistive loss) * 0.4A = 3.8W"
Changed lines of the file:
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@@
   )
   (text "All caps without voltage rating default to 6.3V versions"
-    (at 228.6 15.24 0)
+    (at 139.7 15.24 0)
     (effects (font (size 1.27 1.27) (thickness 0.254) bold) (justify left bottom))
   )
@@
     (effects (font (size 1.27 1.27)) (justify left bottom))
   )
-  (text "Power losses TMC2209:\nFrom datasheet at 1A rms, 24V, Stealth Ploss = 1.4W\nLoss is internal LDO + Drive Stage\nLDO Current output = 7.5mA\n\nat 24V, 1A rms: \nLDO: 24V * 0.0075 = 0.18W\nDrive: (1.4W - 0.18W) / 1 A = 1,22 Ohm\n\nat 16.8V, 0.4A rms: \nLDO: 16.8V * 0.0075 = 0.12W\nDrive: 0.4A² * 1.22 Ohm = 0.19W\n== Loss: 0,3W"
-    (at 228.6 74.93 0)
+  (text "Power losses at TMC2209:\nFrom datasheet at 1A rms, 24V, Stealth Ploss = 1.4W\nLoss is internal LDO + Drive Stage\nLDO Current output = 7.5mA\n\nat 24V, 1A rms: \nLDO: 24V * 0.0075 = 0.18W\nDrive: (1.4W - 0.18W) / 1 A = 1,22 Ohm\n\nat 12V, 1A rms: \nLDO: 12V * 0.0075 = 0.09W\nDrive: 1A² * 1.22 Ohm = 1.22W\n= 1,31W loss at TMC2209\n-----------------------------------"
+    (at 228.6 80.01 0)
     (effects (font (size 1.27 1.27)) (justify left bottom))
   )
@@
     (effects (font (size 1.27 1.27) (thickness 0.254) bold) (justify left bottom))
   )
-  (text "Current (Worst Case):\nBattery low Voltage about 14.7V\nMotor: 3.8W\nDriver: 0.3W\n== Iin = 0.27A\n"
-    (at 228.6 88.9 0)
+  (text "Input Current:\nVoltage about 12V\nMotor: 8.08W\nDriver: 1.31W\n== Iin = (8.08W + 1.31W) / 12V = 0.78A\n"
+    (at 228.6 92.71 0)
     (effects (font (size 1.27 1.27)) (justify left bottom))
   )
-  (text "Stepper motor: 14HY2420\n- used at 0.4 A phase current \n- 20 Ohm coil resistance\n-> 8V, 3.2W resistive losses\n\n- fast rc car servos do up to 80 rpm, 1.3 rps\n- match at least that\n\n- holding torque: 0.12Nm\nBack emf approximation:\n(sqrt(2) * 3.14 * 0.12Nm * 1.3 1/s *) / 0.4A = 1.7V\n\n== (1.7V bemf + 8V resistive loss) * 0.4A = 3.8W "
-    (at 228.6 43.18 0)
+  (text "Power losses at motor:\ncheap Stepper motor 42HB34F1AB-01 as reference:\n- max 1 A phase current \n- 4 Ohm coil resistance\n-> 4V, 4W resistive losses\n\n- tear down: 5\n- revolutions: 2\n- goal time: 2.5 sec\n-> speed (5*2)/2.5 rps = 4 rps\n\n- holding torque: 0.23Nm\nBack emf approximation:\n(sqrt(2) * 3.14 * 0.23Nm * 4 1/s) / 1A = 4.08V\n\n= (4.08V bemf + 4V resistive loss) * 1A \n= 8.08W loss at motor\n-----------------------------------"
+    (at 228.6 49.53 0)
     (effects (font (size 1.27 1.27)) (justify left bottom))
   )
