File: StepperLockingSystem.kicad_sch (KiCad schematic)
At the start: 23 parts, among them J2 DigitalLED, J9 PowerConnector, U3 TC1185, U4 INA180A1

Commit message: Change positions of mounting holes to middle
Parts:
- C4: footprint Capacitor_THT:CP_Radial_D7.5mm_P2.50mm -> Capacitor_THT:CP_Radial_D5.0mm_P2.50mm
Changed lines of the file:
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@@
       (effects (font (size 1.27 1.27)) (justify left))
     )
-    (property "Footprint" "Capacitor_THT:CP_Radial_D7.5mm_P2.50mm" (id 2) (at 74.6252 121.92 0)
+    (property "Footprint" "Capacitor_THT:CP_Radial_D5.0mm_P2.50mm" (id 2) (at 74.6252 121.92 0)
       (effects (font (size 1.27 1.27)) hide)
     )
@@
     )
     (path "/9d62b0fe-2425-4cfb-8192-d872bf181ff2"
-      (reference "C4") (unit 1) (value "180uF") (footprint "Capacitor_THT:CP_Radial_D7.5mm_P2.50mm")
+      (reference "C4") (unit 1) (value "180uF") (footprint "Capacitor_THT:CP_Radial_D5.0mm_P2.50mm")
     )
     (path "/00000000-0000-0000-0000-00005fd04053/a18b8339-d3c7-45ab-98d3-18696f0ed779"
@@
     )
     (path "/00000000-0000-0000-0000-00005fd04053/a1966438-632f-42a0-8f88-339825717af7"
-      (reference "J5") (unit 1) (value "6Pin DuPont 2.56mm") (footprint "Connector_PinHeader_2.54mm:PinHeader_1x06_P2.54mm_Vertical")
+      (reference "J5") (unit 1) (value "6Pin DuPont 2.56mm") (footprint "Connector_PinHeader_2.54mm:PinHeader_2x03_P2.54mm_Vertical")
     )
     (path "/459892de-3652-40e4-b6ee-c2c9debb852e/cd42c423-5e04-46ea-9ad8-3933420402a2"
