File: StepperLockingSystem.kicad_pcb (KiCad board)
At the start: 4 copper layers, 54 x 84 mm, 107 parts, among them J1 signalConnector, J2 digitalLED, J3 6Pin DuPont 2.56mm, J4 SWD, J5 5Pin DuPont 2.54mm, J6 powerConnector, J7 motorNTC, J8 Stepper, J9 hallEncoder, Q1 IRLML0030, SW1 Reset, U1 STM32G0B1KET, U2 24LC64, U3 TC1185, U4 INA180A1, U5 USBLC6-2SC6, U6 USBLC6-2SC6, U7 TMC2209-LA, Y1 ABM3B-16MHz

Commit message: Add settings for Gerber
Other:
- rule pad_to_mask_clearance: 0.05 -> 0
Changed lines of the file:
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@@
       (dielectric_constraints no)
     )
-    (pad_to_mask_clearance 0.05)
-    (solder_mask_min_width 0.254)
+    (pad_to_mask_clearance 0)
     (grid_origin 147.5 135.35)
     (pcbplotparams
       (layerselection 0x00010fc_ffffffff)
       (disableapertmacros false)
-      (usegerberextensions false)
+      (usegerberextensions true)
       (usegerberattributes true)
       (usegerberadvancedattributes true)
@@
       (plotinvisibletext false)
       (sketchpadsonfab false)
-      (subtractmaskfromsilk false)
+      (subtractmaskfromsilk true)
       (outputformat 1)
       (mirror false)
       (drillshape 0)
       (scaleselection 1)
-      (outputdirectory "fab")
+      (outputdirectory "export/gerber")
     )
   )
@@
     (fp_line (start -2.45 -2.35) (end -2.45 3.4) (layer "F.Fab") (width 0.1))
     (fp_line (start 9.95 3.4) (end 9.95 -2.35) (layer "F.Fab") (width 0.1))
-    (pad "1" thru_hole roundrect (at 0 0 180) (size 1.7 1.95) (drill 0.95) (layers *.Cu *.Mask) (roundrect_rratio 0.147059)
+    (pad "1" thru_hole roundrect (at 0 0 180) (size 1.7 1.95) (drill 0.95) (layers *.Cu *.Mask) (roundrect_rratio 0.1470588235)
       (net 14 "/StepperDriver/coilA_2") (pinfunction "Pin_1") (pintype "passive"))
     (pad "2" thru_hole oval (at 2.5 0 180) (size 1.7 1.95) (drill 0.95) (layers *.Cu *.Mask)
@@
     (fp_line (start 0 -2.55) (end -0.5 -3.55) (layer "F.Fab") (width 0.1))
     (fp_line (start 18.78 -4.8) (end -3.54 -4.8) (layer "F.Fab") (width 0.1))
-    (pad "1" thru_hole roundrect (at 0 0 270) (size 2.08 3.6) (drill 1.4) (layers *.Cu *.Mask) (roundrect_rratio 0.120192)
+    (pad "1" thru_hole roundrect (at 0 0 270) (size 2.08 3.6) (drill 1.4) (layers *.Cu *.Mask) (roundrect_rratio 0.1201918269)
       (net 39 "Net-(F1-Pad1)") (pinfunction "Pin_1") (pintype "passive"))
     (pad "2" thru_hole oval (at 5.08 0 270) (size 2.08 3.6) (drill 1.4) (layers *.Cu *.Mask)
@@
     (fp_line (start -1.5 2.5) (end 2.5 2.5) (layer "B.Fab") (width 0.1))
     (fp_line (start -2.5 1.5) (end -1.5 2.5) (layer "B.Fab") (width 0.1))
-    (pad "" smd roundrect (at 0.5 -0.5) (size 0.806226 0.806226) (layers "B.Paste") (roundrect_rratio 0.25))
+    (pad "" smd roundrect (at 0.5 -0.5) (size 0.806226 0.806226) (layers "B.Paste") (roundrect_rratio 0.2500006202))
     (pad "" smd custom (at -1.3375 -1.3375) (size 0.43669 0.43669) (layers "B.Paste")
       (options (clearance outline) (anchor circle))
@@
           ) (width 0.170493) (fill yes))
       ))
-    (pad "" smd roundrect (at -0.5 -0.5) (size 0.806226 0.806226) (layers "B.Paste") (roundrect_rratio 0.25))
+    (pad "" smd roundrect (at -0.5 -0.5) (size 0.806226 0.806226) (layers "B.Paste") (roundrect_rratio 0.2500006202))
     (pad "" smd custom (at 1.3375 -0.5) (size 0.458956 0.458956) (layers "B.Paste")
       (options (clearance outline) (anchor circle))
@@
           ) (width 0.170493) (fill yes))
       ))
-    (pad "" smd roundrect (at -0.5 0.5) (size 0.806226 0.806226) (layers "B.Paste") (roundrect_rratio 0.25))
+    (pad "" smd roundrect (at -0.5 0.5) (size 0.806226 0.806226) (layers "B.Paste") (roundrect_rratio 0.2500006202))
     (pad "" smd custom (at -0.5 -1.3375) (size 0.458956 0.458956) (layers "B.Paste")
       (options (clearance outline) (anchor circle))
@@
           ) (width 0.215024) (fill yes))
       ))
-    (pad "" smd roundrect (at 0.5 0.5) (size 0.806226 0.806226) (layers "B.Paste") (roundrect_rratio 0.25))
+    (pad "" smd roundrect (at 0.5 0.5) (size 0.806226 0.806226) (layers "B.Paste") (roundrect_rratio 0.2500006202))
     (pad "" smd custom (at 1.3375 1.3375) (size 0.43669 0.43669) (layers "B.Paste")
       (options (clearance outline) (anchor circle))
@@
     (fp_line (start 1.6 -0.8) (end -1.6 -0.8) (layer "B.Fab") (width 0.1))
     (fp_line (start -1.6 -0.8) (end -1.6 0.8) (layer "B.Fab") (width 0.1))
-    (pad "1" smd roundrect (at -1.475 0 270) (size 1.15 1.8) (layers "B.Cu" "B.Paste" "B.Mask") (roundrect_rratio 0.217391)
+    (pad "1" smd roundrect (at -1.475 0 270) (size 1.15 1.8) (layers "B.Cu" "B.Paste" "B.Mask") (roundrect_rratio 0.2173913043)
       (net 1 "GND") (pintype "passive"))
-    (pad "2" smd roundrect (at 1.475 0 270) (size 1.15 1.8) (layers "B.Cu" "B.Paste" "B.Mask") (roundrect_rratio 0.217391)
+    (pad "2" smd roundrect (at 1.475 0 270) (size 1.15 1.8) (layers "B.Cu" "B.Paste" "B.Mask") (roundrect_rratio 0.2173913043)
       (net 2 "+3V3") (pintype "passive"))
     (model "${KICAD6_3DMODEL_DIR}/Capacitor_SMD.3dshapes/C_1206_3216Metric.wrl"
@@
     (fp_line (start 1.6 -0.8) (end -1.6 -0.8) (layer "B.Fab") (width 0.1))
     (fp_line (start -1.6 -0.8) (end -1.6 0.8) (layer "B.Fab") (width 0.1))
-    (pad "1" smd roundrect (at -1.475 0 90) (size 1.15 1.8) (layers "B.Cu" "B.Paste" "B.Mask") (roundrect_rratio 0.217391)
+    (pad "1" smd roundrect (at -1.475 0 90) (size 1.15 1.8) (layers "B.Cu" "B.Paste" "B.Mask") (roundrect_rratio 0.2173913043)
       (net 4 "VCC") (pintype "passive"))
-    (pad "2" smd roundrect (at 1.475 0 90) (size 1.15 1.8) (layers "B.Cu" "B.Paste" "B.Mask") (roundrect_rratio 0.217391)
+    (pad "2" smd roundrect (at 1.475 0 90) (size 1.15 1.8) (layers "B.Cu" "B.Paste" "B.Mask") (roundrect_rratio 0.2173913043)
       (net 1 "GND") (pintype "passive"))
     (model "${KICAD6_3DMODEL_DIR}/Capacitor_SMD.3dshapes/C_1206_3216Metric.wrl"
@@
     (fp_line (start -1.6 -0.8) (end -1.6 0.8) (layer "B.Fab") (width 0.1))
     (fp_line (start 1.6 -0.8) (end -1.6 -0.8) (layer "B.Fab") (width 0.1))
-    (pad "1" smd roundrect (at -1.475 0 90) (size 1.15 1.8) (layers "B.Cu" "B.Paste" "B.Mask") (roundrect_rratio 0.217391)
+    (pad "1" smd roundrect (at -1.475 0 90) (size 1.15 1.8) (layers "B.Cu" "B.Paste" "B.Mask") (roundrect_rratio 0.2173913043)
       (net 4 "VCC") (pintype "passive"))
-    (pad "2" smd roundrect (at 1.475 0 90) (size 1.15 1.8) (layers "B.Cu" "B.Paste" "B.Mask") (roundrect_rratio 0.217391)
+    (pad "2" smd roundrect (at 1.475 0 90) (size 1.15 1.8) (layers "B.Cu" "B.Paste" "B.Mask") (roundrect_rratio 0.2173913043)
       (net 1 "GND") (pintype "passive"))
     (model "${KICAD6_3DMODEL_DIR}/Capacitor_SMD.3dshapes/C_1206_3216Metric.wrl"
@@
     (fp_line (start 1 -0.625) (end -1 -0.625) (layer "B.Fab") (width 0.1))
     (fp_line (start -1 0.625) (end 1 0.625) (layer "B.Fab") (width 0.1))
-    (pad "1" smd roundrect (at -0.9125 0 180) (size 1.025 1.4) (layers "B.Cu" "B.Paste" "B.Mask") (roundrect_rratio 0.243902)
+    (pad "1" smd roundrect (at -0.9125 0 180) (size 1.025 1.4) (layers "B.Cu" "B.Paste" "B.Mask") (roundrect_rratio 0.243902439)
       (net 41 "Net-(C29-Pad2)") (pintype "passive"))
-    (pad "2" smd roundrect (at 0.9125 0 180) (size 1.025 1.4) (layers "B.Cu" "B.Paste" "B.Mask") (roundrect_rratio 0.243902)
+    (pad "2" smd roundrect (at 0.9125 0 180) (size 1.025 1.4) (layers "B.Cu" "B.Paste" "B.Mask") (roundrect_rratio 0.243902439)
       (net 1 "GND") (pintype "passive"))
     (model "${KICAD6_3DMODEL_DIR}/Resistor_SMD.3dshapes/R_0805_2012Metric.wrl"
