File: mcu.kicad_sch (KiCad schematic)
At the start: 49 parts, among them J1 signalConnector, J3 6Pin DuPont 2.56mm, J4 SWD, J7 motorNTC, J9 hallEncoder, Q1 IRLML0030, SW1 Reset, U1 STM32G0B1KET, U2 24LC64, U5 USBLC6-2SC6, U6 USBLC6-2SC6, Y1 ABM3B-16MHz

Commit message: Note two known issues
Other:
- note added: "ATTENTION: current LQFP32 doesnt support HSE"
- note added: "ATTENTION: wrong footprint for Mosfet Gate and Source are swapped simply solder Mosfet upside down"
Changed lines of the file:
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@@
     (stroke (width 0) (type default) (color 0 0 0 0))
   )
-  (polyline (pts (xy 257.81 105.41) (xy 257.81 80.01))
+  (polyline (pts (xy 257.81 110.49) (xy 257.81 80.01))
     (stroke (width 0) (type default) (color 0 0 0 0))
   )
@@
     (stroke (width 0) (type default) (color 0 0 0 0))
   )
-  (polyline (pts (xy 214.63 80.01) (xy 214.63 105.41))
+  (polyline (pts (xy 214.63 80.01) (xy 214.63 110.49))
     (stroke (width 0) (type default) (color 0 0 0 0))
   )
@@
     (stroke (width 0) (type default) (color 0 0 0 0))
   )
-  (polyline (pts (xy 214.63 105.41) (xy 257.81 105.41))
+  (polyline (pts (xy 214.63 110.49) (xy 257.81 110.49))
     (stroke (width 0) (type default) (color 0 0 0 0))
   )
@@
   (wire (pts (xy 57.15 31.75) (xy 67.31 31.75))
     (stroke (width 0) (type default) (color 0 0 0 0))
+  )
+  (text "ATTENTION: \nwrong footprint for Mosfet\nGate and Source are swapped\nsimply solder Mosfet upside down\n\n"
+    (at 215.9 69.85 0)
+    (effects (font (size 1.27 1.27) (thickness 0.254) bold italic) (justify left bottom))
   )
   (text "5V tolerant ->" (at 121.92 62.23 180)
@@
   )
   (text "connector for \nmiscellaneous stuff" (at 36.83 130.81 0)
+    (effects (font (size 1.27 1.27) (thickness 0.254) bold italic) (justify left bottom))
+  )
+  (text "ATTENTION:\ncurrent LQFP32 doesnt support HSE" (at 215.9 109.22 0)
     (effects (font (size 1.27 1.27) (thickness 0.254) bold italic) (justify left bottom))
   )
@@
       (effects (font (size 1.27 1.27)) hide)
     )
-    (property "Datasheet" "~" (id 3) (at 246.38 50.8 0)
-      (effects (font (size 1.27 1.27)) hide)
-    )
+    (property "Datasheet" "https://www.infineon.com/dgdl/Infineon-IRLML0030-DataSheet-v01_01-EN.pdf?fileId=5546d462533600a401535664773825df" (id 3) (at 246.38 50.8 0)
+      (effects (font (size 1.27 1.27)) hide)
+    )
