File: signal-splitter/signal-splitter.kicad_pcb (KiCad board)
At the start: 2 copper layers, 36 x 36 mm, 10 parts, among them J1 powerConnector, J2 signalConnector, J3 DoorSwitch, J4 LockSwitch, J5 Buttons, J6 Nerdstern

Commit message: Add settings for Gerber
Changed lines of the file:
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@@
       (layerselection 0x00010fc_ffffffff)
       (disableapertmacros false)
-      (usegerberextensions false)
+      (usegerberextensions true)
       (usegerberattributes true)
       (usegerberadvancedattributes true)
@@
       (plotinvisibletext false)
       (sketchpadsonfab false)
-      (subtractmaskfromsilk false)
+      (subtractmaskfromsilk true)
       (outputformat 1)
       (mirror false)
-      (drillshape 1)
+      (drillshape 0)
       (scaleselection 1)
-      (outputdirectory "")
+      (outputdirectory "export/gerber")
     )
   )
@@
     (fp_line (start 18.78 -2) (end -3.54 -2) (layer "F.Fab") (width 0.1))
     (fp_line (start 18.78 10) (end 18.78 -2) (layer "F.Fab") (width 0.1))
-    (pad "1" thru_hole roundrect (at 0 0 270) (size 2.08 3.6) (drill 1.4) (layers *.Cu *.Mask) (roundrect_rratio 0.120192)
+    (pad "1" thru_hole roundrect (at 0 0 270) (size 2.08 3.6) (drill 1.4) (layers *.Cu *.Mask) (roundrect_rratio 0.1201918269)
       (net 3 "+5V") (pinfunction "Pin_1") (pintype "passive"))
     (pad "2" thru_hole oval (at 5.08 0 270) (size 2.08 3.6) (drill 1.4) (layers *.Cu *.Mask)
